File: EcoSynTech_V6_3_Final.kicad_sch (KiCad schematic)
At the start: 0 parts

Commit message: Add production manufacturing files: real routed Gerber RS-274X, Excellon drill, P&P, fabrication docs
- Real copper trace routing from PCB layout generator (184 traces, 403 vias)
- 215 footprints with accurate pad positions from V3 netlist
- 9 Gerber RS-274X files: F.Cu, B.Cu, F/B.Mask, F/B.Paste, F/B.SilkS, Edge_Cuts
- Excellon drill: 17825 bytes, plated through-hole
- Pick & Place: Top 6325 bytes, Bottom 63 bytes
- Fabrication docs: FABRICATION_NOTES, LAYER_STACKUP, PANELIZATION, GERBER_JOB
Other:
- title: EcoSynTech PCB -> EcoSynTech PCB v6.3
Changed lines of the file:
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@@
+(kicad_sch (version 20230108) (generator "EcoSynTech_PCB_v6.3")
+  (paper "A3")
+  (title_block
+    (title "EcoSynTech PCB v6.3")
+    (company "EcoSynTech Global")
+    (rev "6.3 Final")
+    (date "2026-04-16")
+    (source "EcoSynTech_V6_3_Final")
+    (comment (number 1) (value "Industrial Outdoor IoT Controller"))
+    (comment (number 2) (value "ESP32-WROOM-32E | 2-Layer 200x150mm | ENIG"))
+    (comment (number 3) (value "4+4 Relays | 4+4 Sensors | I2C ADC | USB-UART"))
+    (comment (number 4) (value "Hardware Watchdog | Auto-Reset | Conformal Coating Ready")))
+  (sheet (at 0 0 0) (size 90 45) (sheetname "S01_Power_Input") (sheetfile "S01_Power_Input.kicad_sch"))
+  (sheet (at 0 50 0) (size 90 45) (sheetname "S02_Buck_5V") (sheetfile "S02_Buck_5V.kicad_sch"))
+  (sheet (at 0 100 0) (size 90 45) (sheetname "S03_Buck_3V3") (sheetfile "S03_Buck_3V3.kicad_sch"))
+  (sheet (at 0 150 0) (size 90 45) (sheetname "S04_Rail_Split") (sheetfile "S04_Rail_Split.kicad_sch"))
+  (sheet (at 0 200 0) (size 90 45) (sheetname "S05_OR_Diodes") (sheetfile "S05_OR_Diodes.kicad_sch"))
+  (sheet (at 100 0 0) (size 90 45) (sheetname "S06_ESP32_Core") (sheetfile "S06_ESP32_Core.kicad_sch"))
+  (sheet (at 100 50 0) (size 90 45) (sheetname "S07_USB_UART") (sheetfile "S07_USB_UART.kicad_sch"))
+  (sheet (at 100 100 0) (size 90 45) (sheetname "S08_Watchdog") (sheetfile "S08_Watchdog.kicad_sch"))
+  (sheet (at 100 150 0) (size 90 45) (sheetname "S09_Relay_Drv") (sheetfile "S09_Relay_Drivers.kicad_sch"))
+  (sheet (at 200 0 0) (size 90 45) (sheetname "S10_DHT22") (sheetfile "S10_DHT22.kicad_sch"))
+  (sheet (at 200 50 0) (size 90 45) (sheetname "S11_DS18B20") (sheetfile "S11_DS18B20.kicad_sch"))
+  (sheet (at 200 100 0) (size 90 45) (sheetname "S12_Soil_Sensor") (sheetfile "S12_Soil_Sensor.kicad_sch"))
+  (sheet (at 200 150 0) (size 90 45) (sheetname "S13_VIN_Sense") (sheetfile "S13_VIN_Sense.kicad_sch"))
+  (sheet (at 200 200 0) (size 90 45) (sheetname "S14_ADS1115") (sheetfile "S14_ADS1115.kicad_sch"))
+  (sheet (at 300 0 0) (size 90 45) (sheetname "S15_I2C_Bus") (sheetfile "S15_I2C_Bus.kicad_sch"))
+  (sheet (at 300 50 0) (size 90 45) (sheetname "S16_MicroSD") (sheetfile "S16_MicroSD.kicad_sch"))
+  (sheet (at 300 100 0) (size 90 45) (sheetname "S17_IO_Expnd") (sheetfile "S17_IO_Expanders.kicad_sch"))
+  (sheet (at 300 150 0) (size 90 45) (sheetname "S18_Exp_Relays") (sheetfile "S18_Exp_Relays.kicad_sch"))
+  (sheet (at 300 200 0) (size 90 45) (sheetname "S19_Debug_TP") (sheetfile "S19_Debug.kicad_sch"))
+  (sheet (at 300 250 0) (size 90 45) (sheetname "S20_Ext_Conn") (sheetfile "S20_External_Conn.kicad_sch"))
+)
