File: EcoSynTech_V6_3_Final.kicad_pcb (KiCad board)
At the start: 2 copper layers, 0 parts

Commit message: Add production manufacturing files: real routed Gerber RS-274X, Excellon drill, P&P, fabrication docs
- Real copper trace routing from PCB layout generator (184 traces, 403 vias)
- 215 footprints with accurate pad positions from V3 netlist
- 9 Gerber RS-274X files: F.Cu, B.Cu, F/B.Mask, F/B.Paste, F/B.SilkS, Edge_Cuts
- Excellon drill: 17825 bytes, plated through-hole
- Pick & Place: Top 6325 bytes, Bottom 63 bytes
- Fabrication docs: FABRICATION_NOTES, LAYER_STACKUP, PANELIZATION, GERBER_JOB
Parts:
- added ?: , CONN_5.08_2P,  at (10.0, 18.0)
- added ?: , R_0805,  at (105.0, 5.00)
- added ?: , SOT-23,  at (140.0, 93.0)
- added ?: , SOT-23,  at (148.0, 110.0)
- added ?: , R_0805,  at (155.0, 110.0)
- added ?: , D_SOD-123,  at (167.0, 110.0)
- added ?: , SOT-23,  at (140.0, 110.0)
- added ?: , SOT-23,  at (148.0, 127.0)
- added ?: , R_0805,  at (155.0, 127.0)
- added ?: , D_SOD-123,  at (167.0, 127.0)
- added ?: , SOT-23,  at (140.0, 127.0)
- added ?: , SOT-23,  at (148.0, 144.0)
- added ?: , D_SOD-123,  at (105.0, 27.0)
- added ?: , R_0805,  at (155.0, 144.0)
- added ?: , D_SOD-123,  at (167.0, 144.0)
- added ?: , SOT-23,  at (140.0, 144.0)
- added ?: , RELAY_SRD_5V,  at (175.0, 93.0)
- added ?: , CONN_7.62_3P,  at (185.0, 93.0)
- added ?: , RELAY_SRD_5V,  at (175.0, 110.0)
- added ?: , CONN_7.62_3P,  at (185.0, 110.0)
- added ?: , RELAY_SRD_5V,  at (175.0, 127.0)
- added ?: , CONN_7.62_3P,  at (185.0, 127.0)
- added ?: , RELAY_SRD_5V,  at (175.0, 144.0)
- added ?: , CAP_D8x11.5,  at (120.0, 18.0)
- added ?: , CONN_7.62_3P,  at (185.0, 144.0)
- added ?: , SOT-23,  at (45.0, 93.0)
- added ?: , SOT-23,  at (55.0, 93.0)
- added ?: , R_0805,  at (65.0, 93.0)
- added ?: , R_0805,  at (65.0, 88.0)
- added ?: , DHT22_TH,  at (50.0, 45.0)
- added ?: , CONN_3.81_3P,  at (40.0, 35.0)
- added ?: , R_0805,  at (48.0, 38.0)
- added ?: , D_SOD-123,  at (55.0, 40.0)
- added ?: , TO-92,  at (50.0, 55.0)
- added ?: , C_1210,  at (130.0, 12.0)
- added ?: , CONN_3.81_3P,  at (40.0, 45.0)
- added ? (x2): , R_0805,  at (48.0, 48.0)
- added ?: , D_SOD-123,  at (55.0, 50.0)
- added ?: , MSOP-8,  at (82.0, 53.0)
- added ?: , C_0805,  at (87.0, 57.0)
- added ?: , C_0805,  at (90.0, 57.0)
- added ?: , R_0805,  at (75.0, 48.0)
- added ?: , D_SOD-123,  at (78.0, 48.0)
- added ?: , R_0805,  at (78.0, 48.0)
- added ?: , D_SOD-123,  at (81.0, 48.0)
- added ?: , C_0805,  at (130.0, 23.0)
- added ?: , R_0805,  at (81.0, 48.0)
- added ?: , D_SOD-123,  at (84.0, 48.0)
- added ?: , R_0805,  at (84.0, 48.0)
- added ?: , D_SOD-123,  at (87.0, 48.0)
- added ?: , CONN_3.81_6P,  at (112.5, 60.0)
- added ?: , CONN_5.08_2P,  at (190.0, 28.0)
- added ?: , R_0805,  at (178.0, 28.0)
- added ?: , R_0805,  at (175.0, 25.0)
- added ?: , C_0805,  at (178.0, 22.0)
- added ?: , R_0805,  at (173.0, 28.0)
- added ?: , SOIC-8E,  at (72.0, 35.0)
- added ?: , SOT-23,  at (170.0, 28.0)
- added ?: , CONN_3.81_3P,  at (40.0, 55.0)
- added ?: , R_0805,  at (35.0, 55.0)
- added ?: , C_0805,  at (32.0, 55.0)
- added ?: , D_SOD-123,  at (29.0, 55.0)
- added ?: , CONN_3.81_4P,  at (35.0, 23.0)
- added ?: , CONN_3.81_4P,  at (35.0, 25.0)
- added ?: , R_0805,  at (60.0, 43.0)
- added ?: , R_0805,  at (60.0, 48.0)
- added ?: , R_0805,  at (48.0, 43.0)
- added ?: , C_1210,  at (60.0, 42.0)
- added ?: , D_SOD-123,  at (43.0, 43.0)
- added ?: , D_SOD-123,  at (43.0, 48.0)
- added ?: , BME280_I2C,  at (127.5, 55.0)
- added ?: , OLED_I2C,  at (145.0, 55.0)
- added ?: , MICROSD,  at (140.0, 80.0)
- added ?: , R_0805,  at (134.0, 83.0)
- added ?: , R_0805,  at (134.0, 80.0)
- added ?: , R_0805,  at (134.0, 77.0)
- added ?: , R_0805,  at (134.0, 74.0)
- added ?: , C_0805,  at (60.0, 35.0)
- added ?: , R_0805,  at (134.0, 71.0)
- added ?: , C_0805,  at (137.0, 83.0)
- added ?: , SSOP-28,  at (50.0, 110.0)
- added ?: , SSOP-28,  at (50.0, 125.0)
- added ?: , C_0805,  at (105.0, 115.0)
- added ?: , C_0805,  at (108.0, 115.0)
- added ?: , C_0805,  at (120.0, 130.0)
- added ?: , C_0805,  at (123.0, 130.0)
- added ?: , SOT-23,  at (62.0, 93.0)
- added ?: , R_0805,  at (55.0, 93.0)
- added ?: , L_6x6,  at (83.0, 35.0)
- added ?: , D_SOD-123,  at (48.0, 93.0)
- added ?: , SOT-23,  at (62.0, 110.0)
- added ?: , R_0805,  at (55.0, 110.0)
- added ?: , D_SOD-123,  at (48.0, 110.0)
- added ?: , SOT-23,  at (62.0, 127.0)
- added ?: , R_0805,  at (55.0, 127.0)
- added ?: , D_SOD-123,  at (48.0, 127.0)
- added ?: , SOT-23,  at (62.0, 144.0)
- added ?: , R_0805,  at (55.0, 144.0)
- added ?: , D_SOD-123,  at (48.0, 144.0)
- added ?: , C_1210,  at (93.0, 42.0)
- added ?: , TESTPOINT,  at (5.00, 0.00)
- added ?: , TESTPOINT,  at (5.00, 3.00)
- added ?: , TESTPOINT,  at (5.00, 6.00)
- added ?: , TESTPOINT,  at (5.00, 9.00)
- added ?: , TESTPOINT,  at (5.00, 12.0)
- added ?: , TESTPOINT,  at (5.00, 15.0)
- added ?: , TESTPOINT,  at (5.00, 18.0)
- added ?: , TESTPOINT,  at (5.00, 21.0)
- added ?: , TESTPOINT,  at (5.00, 24.0)
- added ?: , TESTPOINT,  at (5.00, 27.0)
- added ?: , FUSE_HOLDER_5x20,  at (22.0, 18.0)
- added ?: , C_1210,  at (93.0, 38.0)
- added ?: , TESTPOINT,  at (5.00, 30.0)
- added ?: , TESTPOINT,  at (5.00, 33.0)
- added ?: , TESTPOINT,  at (5.00, 36.0)
- added ?: , TESTPOINT,  at (5.00, 39.0)
- added ?: , TESTPOINT,  at (5.00, 42.0)
- added ?: , TESTPOINT,  at (5.00, 45.0)
- added ?: , CONN_7.62_2P,  at (190.0, 20.0)
- added ?: , CONN_5.08_2x5,  at (90.0, 42.5)
- added ?: , SOT-23,  at (75.0, 40.0)
- added ?: , SOT-23,  at (75.0, 44.0)
- added ?: , C_0805,  at (93.0, 34.0)
- added ?: , SOT-23,  at (75.0, 48.0)
- added ?: , SOT-23,  at (75.0, 52.0)
- added ?: , M3_HOLE,  at (5.00, 5.00)
- added ?: , M3_HOLE,  at (5.00, 145.0)
- added ?: , M3_HOLE,  at (195.0, 5.00)
- added ?: , M3_HOLE,  at (195.0, 145.0)
- added ?: , R_0805,  at (82.0, 28.0)
- added ?: , R_0805,  at (82.0, 24.0)
- added ?: , R_0805,  at (60.0, 28.0)
- added ?: , D_SMA,  at (90.0, 50.0)
- added ?: , VIA,  at (68.0, 38.0)
- added ?: , VIA,  at (68.0, 35.0)
- added ?: , VIA,  at (68.0, 32.0)
- added ?: , VIA,  at (76.0, 38.0)
- added ?: , GDT,  at (35.0, 18.0)
- added ?: , VIA,  at (76.0, 35.0)
- added ?: , VIA,  at (76.0, 32.0)
- added ?: , SOIC-8E,  at (112.0, 35.0)
- added ?: , C_1210,  at (100.0, 42.0)
- added ?: , C_0805,  at (100.0, 35.0)
- added ?: , L_6x6,  at (123.0, 35.0)
- added ?: , C_1210,  at (133.0, 42.0)
- added ?: , C_1210,  at (133.0, 38.0)
- added ?: , C_0805,  at (133.0, 34.0)
- added ?: , R_0805,  at (122.0, 28.0)
- added ?: , MOV,  at (48.0, 18.0)
- added ?: , R_0805,  at (122.0, 24.0)
- added ?: , R_0805,  at (100.0, 28.0)
- added ?: , VIA,  at (108.0, 38.0)
- added ?: , VIA,  at (108.0, 35.0)
- added ?: , VIA,  at (108.0, 32.0)
- added ?: , VIA,  at (116.0, 38.0)
- added ?: , VIA,  at (116.0, 35.0)
- added ?: , VIA,  at (116.0, 32.0)
- added ?: , FB_0805,  at (58.0, 47.0)
- added ?: , C_0805,  at (63.0, 47.0)
- added ?: , R_2512,  at (62.0, 18.0)
- added ?: , C_0805,  at (66.0, 47.0)
- added ?: , FB_0805,  at (58.0, 67.0)
- added ?: , C_0805,  at (63.0, 67.0)
- added ?: , C_0805,  at (66.0, 67.0)
- added ?: , SOT-23,  at (138.0, 57.0)
- added ?: , C_0805,  at (141.0, 57.0)
- added ?: , D_SMA,  at (20.0, 35.0)
- added ?: , D_SMA,  at (27.0, 35.0)
- added ?: , C_1210,  at (35.0, 35.0)
- added ?: , C_0805,  at (40.0, 35.0)
- added ?: , INDUCTOR,  at (75.0, 18.0)
- added ?: , ESP32-WROOM-32E,  at (165.0, 57.5)
- added ?: , C_0805,  at (150.0, 70.0)
- added ?: , C_0805,  at (152.0, 73.0)
- added ?: , C_0805,  at (154.0, 76.0)
- added ?: , R_0805,  at (160.0, 68.0)
- added ?: , R_0805,  at (163.0, 68.0)
- added ?: , R_0805,  at (166.0, 68.0)
- added ?: , LED_0805,  at (155.0, 50.0)
- added ?: , R_0805,  at (152.0, 50.0)
- added ?: , LED_0805,  at (155.0, 53.0)
- added ?: , D_SMB,  at (90.0, 18.0)
- added ?: , R_0805,  at (152.0, 53.0)
- added ?: , LED_0805,  at (155.0, 56.0)
- added ?: , R_0805,  at (152.0, 56.0)
- added ?: , LED_0805,  at (155.0, 59.0)
- added ?: , R_0805,  at (152.0, 59.0)
- added ?: , R_0805,  at (40.0, 45.0)
- added ?: , R_0805,  at (40.0, 55.0)
- added ?: , R_0805,  at (170.0, 72.0)
- added ?: , USB_MICRO_B,  at (25.0, 30.0)
- added ?: , FUSE_PTC,  at (32.0, 30.0)
- added ?: , SO-8,  at (105.0, 18.0)
- added ?: , D_SMB,  at (39.0, 30.0)
- added ?: , R_1206,  at (46.0, 30.0)
- added ?: , SOT-23-6,  at (53.0, 30.0)
- added ?: , QFN-28,  at (35.0, 53.0)
- added ?: , SOT-23,  at (40.0, 60.0)
- added ?: , R_0805,  at (37.0, 60.0)
- added ?: , SOT-23,  at (40.0, 65.0)
- added ?: , R_0805,  at (37.0, 65.0)
- added ?: , SOT-23-6,  at (50.0, 58.0)
- added ?: , R_0805,  at (58.0, 58.0)
- added ?: , R_0805,  at (105.0, 10.0)
- added ?: , R_0805,  at (47.0, 61.0)
- added ?: , R_0805,  at (55.0, 61.0)
- added ?: , C_0805,  at (50.0, 64.0)
- added ?: , SOT-23,  at (55.0, 60.0)
- added ?: , R_2512,  at (15.0, 88.0)
- added ?: , CAP_D10x12.5,  at (28.0, 88.0)
- added ?: , D_SMB,  at (40.0, 88.0)
- added ?: , SOT-23,  at (148.0, 93.0)
- added ?: , R_0805,  at (155.0, 93.0)
- added ?: , D_SOD-123,  at (167.0, 93.0)
Routing:
- net 26: track 0.00 -> 31668803.9 mm
- net 27: track 0.00 -> 29013493.9 mm
- net 24: track 0.00 -> 15420000.0 mm
- net 38: track 0.00 -> 14708011.0 mm
- net 25: track 0.00 -> 14410000.0 mm
- net 39: track 0.00 -> 12740000.0 mm
- net 30: track 0.00 -> 12360000.0 mm
- net 43: track 0.00 -> 9500000.0 mm
- net 37: track 0.00 -> 8818000.0 mm
- net 36: track 0.00 -> 7372000.0 mm
- net 48: track 0.00 -> 6670000.0 mm, vias 0 -> 2
- net 11: track 0.00 -> 6352610.9 mm
- net 35: track 0.00 -> 5926000.0 mm
- net 47: track 0.00 -> 5040000.0 mm, vias 0 -> 2
- net 40: track 0.00 -> 5000000.0 mm
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- added copper zone on B.Cu, net GND_STAR
- added copper zone on F.Cu, net GND_STAR
Other:
- rule pad_to_mask_clearance: 0.0 -> 0.05
- board text added: "2026-04-16"
- board text added: "ANTENNA KEEPOUT ZONE"
- board text added: "CAUTION: HIGH VOLTAGE 220VAC"
- board text added: "DO NOT REMOVE SNUBBER - ARC HAZARD"
- board text added: "EcoSynTech Global | ecosyntech68vn"
- board text added: "EcoSynTech V6.3 Industrial Pro"
- board text added: "KIEM TRA CUC TINH TRUOC KHI CAP NGUON"
- board text added: "Rev 6.3 Final | 2-Layer | ENIG | FR-4 Tg130"
- board text added: "THAY DUNG GIA TRI CAU CHI"

Commit message: Fix manufacturing files: METRIC drill format, add RELAY5-8, 223 footprints, complete Gerber RS-274X
Bugs fixed:
- Drill file: INCH,TZ → METRIC,TZ (was breaking CAM tools)
- Added missing RELAY5-8 and J_R5-8 footprints (expansion relays)
- Added relay coil traces for RELAY1-8 and Q_R5-8 drivers

PCB: 223 footprints, 221 copper traces, 405 vias
Manufacturing: 644 components (incl. thermal/GND stitching)
P&P Top: 313 components
F.Cu: 83KB, B.Cu: 40KB, Drill: 22KB

Also: Add generator scripts (gen_pcb_v2.py, gen_mfg_v2.py, components_gen.py)
Parts:
- removed the ? at (148.0, 110.0)
- removed the ? at (155.0, 110.0)
- removed the ? at (148.0, 127.0)
- removed the ? at (155.0, 127.0)
- removed the ? at (148.0, 144.0)
- removed the ? at (155.0, 144.0)
- removed the ? at (48.0, 48.0) (x2)
- removed the ? at (62.0, 93.0)
- removed the ? at (55.0, 93.0)
- removed the ? at (48.0, 93.0)
- removed the ? at (62.0, 110.0)
- removed the ? at (55.0, 110.0)
- removed the ? at (48.0, 110.0)
- removed the ? at (62.0, 127.0)
- removed the ? at (55.0, 127.0)
- removed the ? at (48.0, 127.0)
- removed the ? at (62.0, 144.0)
- removed the ? at (55.0, 144.0)
- removed the ? at (48.0, 144.0)
- removed the ? at (148.0, 93.0)
- removed the ? at (155.0, 93.0)
- added ? (x2): , SOT-23,  at (148.0, 110.0)
- added ? (x2): , R_0805,  at (155.0, 110.0)
- added ? (x2): , SOT-23,  at (148.0, 127.0)
- added ? (x2): , R_0805,  at (155.0, 127.0)
- added ? (x2): , SOT-23,  at (148.0, 144.0)
- added ? (x2): , R_0805,  at (155.0, 144.0)
- added ? (x2): , R_0805,  at (48.0, 48.0)
- added ? (x2): , SOT-23,  at (148.0, 93.0)
- added ? (x2): , R_0805,  at (155.0, 93.0)
- added ?: , D_SOD-123,  at (162.0, 93.0)
- added ?: , RELAY_SRD_5V,  at (168.0, 93.0)
- added ?: , CONN_7.62_3P,  at (178.0, 93.0)
- added ?: , D_SOD-123,  at (162.0, 110.0)
- added ?: , RELAY_SRD_5V,  at (168.0, 110.0)
- added ?: , CONN_7.62_3P,  at (178.0, 110.0)
- added ?: , D_SOD-123,  at (162.0, 127.0)
- added ?: , RELAY_SRD_5V,  at (168.0, 127.0)
- added ?: , CONN_7.62_3P,  at (178.0, 127.0)
- added ?: , D_SOD-123,  at (162.0, 144.0)
- added ?: , RELAY_SRD_5V,  at (168.0, 144.0)
- added ?: , CONN_7.62_3P,  at (178.0, 144.0)
Routing:
- net 8: track 2500000.0 -> 51236070.5 mm
- net 1: track 0.00 -> 12832000.0 mm
- net 48: track 6670000.0 -> 15270000.0 mm
- net 47: track 5040000.0 -> 13640000.0 mm
- net 46: track 3410000.0 -> 12010000.0 mm
- net 45: track 4620000.0 -> 13220000.0 mm
